File: CNCPlotter.sch (EAGLE design)
At the start: 125 parts, among them IC1 HEF4050B, IC2 MC34063, IC3 LD1117S33, IC4 74HC4094, IC5 ATmega32U4, IC6 DRV8811, IC7 DRV8811, J1 Home Switches, J10 ISP, J11 X Motor, J12 MS1, J13 MS0, J14 Y Motor, J15 MS1, J16 MS0, J2 Touchscreen, J3 12V Supply, J4 MicroSD Card, J5 HWB, J6 USB-FT, J7 Servo, J8 Z Drive, J9 UART, Q1 16MHz

Commit message: foo
Connections:
- removed net N$71: R42.2, VR3.E
- net N$20: now also R42.2, VR3.A
- net N$60: now also VR2.E; no longer VR2.A
- net N$61: now also VR2.A; no longer VR2.E
- net N$70: now also VR3.E; no longer VR3.A
Other:
- moved on the sheet: VR2, VR3
Changed lines of the file:
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@@
 <text x="55.88" y="53.34" size="1.27" layer="98">0603</text>
 <text x="63.5" y="53.34" size="1.27" layer="98">0603</text>
-<text x="55.88" y="83.82" size="1.27" layer="98">0603</text>
+<text x="53.34" y="86.36" size="1.27" layer="98">0603</text>
 <text x="45.72" y="73.66" size="1.27" layer="98">CT6EP103-ND</text>
 <text x="76.2" y="78.74" size="1.27" layer="98">0603</text>
@@
 <attribute name="VALUE" x="20.32" y="243.84" size="1.27" layer="96"/>
 </instance>
-<instance part="VR2" gate="1" x="60.96" y="266.7" smashed="yes" rot="MR180">
+<instance part="VR2" gate="1" x="60.96" y="266.7" smashed="yes">
 <attribute name="NAME" x="53.34" y="266.7" size="1.27" layer="95"/>
 <attribute name="VALUE" x="53.34" y="264.16" size="1.27" layer="96"/>
@@
 <attribute name="VALUE" x="20.32" y="55.88" size="1.27" layer="96"/>
 </instance>
-<instance part="VR3" gate="1" x="60.96" y="78.74" smashed="yes" rot="MR180">
-<attribute name="NAME" x="53.34" y="78.74" size="1.27" layer="95"/>
-<attribute name="VALUE" x="53.34" y="76.2" size="1.27" layer="96"/>
+<instance part="VR3" gate="1" x="60.96" y="78.74" smashed="yes">
+<attribute name="NAME" x="58.42" y="78.74" size="1.27" layer="95" rot="MR0"/>
+<attribute name="VALUE" x="58.42" y="76.2" size="1.27" layer="96" rot="MR0"/>
 </instance>
 <instance part="R46" gate="G$1" x="187.96" y="60.96" smashed="yes" rot="R90">
@@
 </instance>
 <instance part="R38" gate="G$1" x="60.96" y="91.44" smashed="yes" rot="R90">
-<attribute name="NAME" x="55.88" y="88.9" size="1.27" layer="95"/>
-<attribute name="VALUE" x="55.88" y="86.36" size="1.27" layer="96"/>
+<attribute name="NAME" x="53.34" y="91.44" size="1.27" layer="95"/>
+<attribute name="VALUE" x="53.34" y="88.9" size="1.27" layer="96"/>
 </instance>
 <instance part="R39" gate="G$1" x="81.28" y="83.82" smashed="yes" rot="R90">
@@
 </segment>
 </net>
-<net name="N$60" class="0">
-<segment>
-<wire x1="60.96" y1="274.32" x2="60.96" y2="271.78" width="0.1524" layer="91"/>
-<pinref part="VR2" gate="1" pin="A"/>
-<pinref part="R24" gate="G$1" pin="1"/>
-</segment>
-</net>
-<net name="N$61" class="0">
-<segment>
-<wire x1="60.96" y1="261.62" x2="60.96" y2="254" width="0.1524" layer="91"/>
-<pinref part="VR2" gate="1" pin="E"/>
-<pinref part="R28" gate="G$1" pin="2"/>
-</segment>
-</net>
 <net name="N$64" class="0">
 <segment>
 <pinref part="IC6" gate="G$1" pin="VREF"/>
-<wire x1="63.5" y1="266.7" x2="68.58" y2="266.7" width="0.1524" layer="91"/>
 <wire x1="68.58" y1="266.7" x2="71.12" y2="264.16" width="0.1524" layer="91"/>
 <wire x1="71.12" y1="264.16" x2="147.32" y2="264.16" width="0.1524" layer="91"/>
 <wire x1="71.12" y1="251.46" x2="71.12" y2="264.16" width="0.1524" layer="91"/>
 <junction x="71.12" y="264.16"/>
+<pinref part="C19" gate="G$1" pin="1"/>
 <pinref part="VR2" gate="1" pin="S"/>
-<pinref part="C19" gate="G$1" pin="1"/>
+<wire x1="63.5" y1="266.7" x2="68.58" y2="266.7" width="0.1524" layer="91"/>
 </segment>
 </net>
@@
 <segment>
 <pinref part="IC7" gate="G$1" pin="RCB"/>
-<wire x1="147.32" y1="68.58" x2="50.8" y2="68.58" width="0.1524" layer="91"/>
+<wire x1="147.32" y1="68.58" x2="60.96" y2="68.58" width="0.1524" layer="91"/>
+<wire x1="60.96" y1="68.58" x2="50.8" y2="68.58" width="0.1524" layer="91"/>
 <wire x1="50.8" y1="68.58" x2="38.1" y2="68.58" width="0.1524" layer="91"/>
 <wire x1="38.1" y1="68.58" x2="38.1" y2="66.04" width="0.1524" layer="91"/>
@@
 <pinref part="C30" gate="G$1" pin="1"/>
 <wire x1="50.8" y1="63.5" x2="50.8" y2="68.58" width="0.1524" layer="91"/>
+<pinref part="VR3" gate="1" pin="A"/>
+<pinref part="R42" gate="G$1" pin="2"/>
+<wire x1="60.96" y1="73.66" x2="60.96" y2="68.58" width="0.1524" layer="91"/>
+<wire x1="60.96" y1="66.04" x2="60.96" y2="68.58" width="0.1524" layer="91"/>
 </segment>
 </net>
@@
 </segment>
 </net>
-<net name="N$70" class="0">
-<segment>
-<wire x1="60.96" y1="86.36" x2="60.96" y2="83.82" width="0.1524" layer="91"/>
-<pinref part="VR3" gate="1" pin="A"/>
-<pinref part="R38" gate="G$1" pin="1"/>
-</segment>
-</net>
-<net name="N$71" class="0">
-<segment>
-<wire x1="60.96" y1="73.66" x2="60.96" y2="66.04" width="0.1524" layer="91"/>
-<pinref part="VR3" gate="1" pin="E"/>
-<pinref part="R42" gate="G$1" pin="2"/>
-</segment>
-</net>
 <net name="N$72" class="0">
 <segment>
 <pinref part="IC7" gate="G$1" pin="VREF"/>
-<wire x1="63.5" y1="78.74" x2="68.58" y2="78.74" width="0.1524" layer="91"/>
-<wire x1="68.58" y1="78.74" x2="71.12" y2="76.2" width="0.1524" layer="91"/>
 <wire x1="71.12" y1="76.2" x2="147.32" y2="76.2" width="0.1524" layer="91"/>
 <wire x1="71.12" y1="63.5" x2="71.12" y2="76.2" width="0.1524" layer="91"/>
 <junction x="71.12" y="76.2"/>
+<pinref part="C31" gate="G$1" pin="1"/>
 <pinref part="VR3" gate="1" pin="S"/>
-<pinref part="C31" gate="G$1" pin="1"/>
+<wire x1="71.12" y1="76.2" x2="68.58" y2="78.74" width="0.1524" layer="91"/>
+<wire x1="68.58" y1="78.74" x2="63.5" y2="78.74" width="0.1524" layer="91"/>
 </segment>
 </net>
@@
 </segment>
 </net>
+<net name="N$60" class="0">
+<segment>
+<pinref part="R24" gate="G$1" pin="1"/>
+<pinref part="VR2" gate="1" pin="E"/>
+<wire x1="60.96" y1="274.32" x2="60.96" y2="271.78" width="0.1524" layer="91"/>
+</segment>
+</net>
+<net name="N$61" class="0">
+<segment>
+<pinref part="VR2" gate="1" pin="A"/>
+<pinref part="R28" gate="G$1" pin="2"/>
+<wire x1="60.96" y1="261.62" x2="60.96" y2="254" width="0.1524" layer="91"/>
+</segment>
+</net>
+<net name="N$70" class="0">
+<segment>
+<pinref part="R38" gate="G$1" pin="1"/>
+<pinref part="VR3" gate="1" pin="E"/>
+<wire x1="60.96" y1="86.36" x2="60.96" y2="83.82" width="0.1524" layer="91"/>
+</segment>
+</net>

Commit message: foo
Parts:
- added J17: MS0, freetronics-luke:SJ
- C1, C13, C25: value 100 uF -> 100uF
- C10, C7, C8: value 100nF -> 100 nF; device freetronics:CAP0603 -> freetronics-master-v1:CAP0603
- C11, C12: device freetronics:CAP0603 -> freetronics-master-v1:CAP0603
- C17, C18, C29, C30: value 680 pF -> 1nF
- C9: value 1uF -> 1 uF; device freetronics:CAP0603 -> freetronics-master-v1:CAP0603
- F1: value 500mA PPTC -> 500mA
- J1: value Home Switches -> Servo; device con-molex:22-23-2061 -> con-molex:22-23-2031
- J10: value ISP -> Touchscreen; device SparkFun:AVR_SPI_PRG_6NS -> pinhead:PINHD-1X4
- J11: value X Motor -> Touchscreen; device con-phoenix-254:MPT4 -> SparkFun:DS_TOUCH_CONNECTOR; OC_FARNELL unknown -> (none); OC_NEWARK unknown -> (none)
- J12: value MS1 -> X Motor; device freetronics-luke:SJ -> con-phoenix-254:MPT4; OC_FARNELL (none) -> unknown; OC_NEWARK (none) -> unknown
- J13, J16: value MS0 -> MS1
- J14: value Y Motor -> MS0; device con-phoenix-254:MPT4 -> freetronics-luke:SJ; OC_FARNELL unknown -> (none); OC_NEWARK unknown -> (none)
- J15: value MS1 -> Y Motor; device freetronics-luke:SJ -> con-phoenix-254:MPT4; OC_FARNELL (none) -> unknown; OC_NEWARK (none) -> unknown
- J2: value Touchscreen -> Z Drive; device SparkFun:DS_TOUCH_CONNECTOR -> con-phoenix-254:MPT5
- J3: value 12V Supply -> ISP; device SparkFun:POWER_JACKSLT -> SparkFun:AVR_SPI_PRG_6NS
- J4: value MicroSD Card -> UART; device RAMPSdisplay:ADAFRUIT_MICROSD -> pinhead:PINHD-1X4
- J5: value HWB -> 12V Supply; device freetronics-luke:SJ -> SparkFun:POWER_JACKSLT
- J6: value USB-FT -> MicroSD Card; device freetronics-luke:USB-FT -> RAMPSdisplay:ADAFRUIT_MICROSD
- J7: value Servo -> HWB; device con-molex:22-23-2031 -> freetronics-luke:SJ
- J8: value Z Drive -> USB-FT; device con-molex:22-23-2051 -> freetronics-luke:USB-FT
- J9: value UART -> Home Switches; device con-molex:22-23-2041 -> con-phoenix-254:MPT6
- LED1: value TXD -> TX
- LED2: value RXD -> RX
- LED4: value Z Home -> Z
- LED5: value Y Home -> Y
- LED6: value X Home -> X
- LED7: value 12V -> 12
- R10: value 10k -> 3k0
- R11: value 0.2 ohms -> 1k; device rcl:R-EU_R1210 -> freetronics-master-v1:RESISTOR0603
- R12: value 1k -> 22R
- R13: value 3k0 -> 10k
- R14: value 1k -> 10k
- R16: value 10k -> 22R
- R18, R19: value 22R -> 10k
- R20, R21, R22, R23, R25, R30, R31: value 10k -> 10K
- R24: value 3k3 -> 3K3
- R26, R27, R40, R41: value 56k -> 47K
- R29, R43: value 4k7 -> 4K7
- R32, R33: value 0.2R 1W -> 0.25R 1W
- R8: value 10k -> 0.2 ohms; device freetronics-master-v1:RESISTOR0603 -> rcl:R-EU_R1210
- R9: value 10k -> 1k
- VR2: value 10 k -> 10K
Connections:
- new net N$71: R42.2, VR3.A
- net !RESET: now also J3.5, R14.1; no longer J10.5, R17.1
- net !SD_CS: now also R13.1; no longer R16.1
- net +12V: now also J2-1.1, J5.PWR, R8.1; no longer J3.PWR, J8-1.S, R11.1
- net +5V: now also J1-2.S, J2-3.1, J3.2, J4.1, J9-1.1, J9-3.1, J9-5.1, R12.2, R13.2, R14.2; no longer J1-1.S, J1-3.S, J1-5.S, J10.2, J7-2.S, J8-3.S, J9-1.S, R15.2, R16.2, R17.2
- net FOO: now also J6.CS; no longer J4.CS
- net GND: now also C7.2, J1-1.S, J14.1, J17.1, J2-2.1, J3.6, J4.2, J5.GND, J6.GND1, J6.VSS, J7.1, J8.GND, J8.SH$1, R17.2, R18.2, R19.2; no longer C7.1, J10.6, J12.1, J15.1, J3.GNDBREAK, J4.GND, J4.GND1, J4.VSS, J5.1, J6.SH$1, J7-1.S, J8-2.S, J9-2.S, R10.2, R12.2, R8.2
- net HWB: now also J7.2; no longer J5.2
- net MISO: now also J3.1, J6.DATA_OUT; no longer J10.1, J4.DATA_OUT
- net MOSI: now also J3.4; no longer J10.4
- net MOSI_3.3V: now also J6.DATA_IN; no longer J4.DATA_IN
- net N$1: now also J15-1.1; no longer J14-1.1
- net N$2: now also J8.VBUS; no longer J6.VBUS
- net N$20: no longer R42.2, VR3.A
- net N$21: now also J12-4.1; no longer J11-4.1
- net N$22: now also J12-3.1; no longer J11-3.1
- net N$23: now also J12-2.1; no longer J11-2.1
- net N$3: now also J12-1.1; no longer J11-1.1
- net N$32: now also R8.2; no longer R11.2
- net N$33: now also J8.D+, R16.2; no longer J6.D+, R19.2
- net N$34: now also J8.D-, R15.2; no longer J6.D-, R18.2
- net N$37: now also R16.1; no longer R19.1
- net N$38: now also R15.1; no longer R18.1
- net N$4: now also J15-4.1; no longer J14-4.1
- net N$40: now also C7.1; no longer C7.2
- net N$44: now also R10.2, R9.1; no longer R12.1, R13.2
- net N$5: now also J15-3.1; no longer J14-3.1
- net N$59: now also R12.1; no longer R15.1
- net N$6: now also J15-2.1; no longer J14-2.1
- net N$62: now also R11.1; no longer R14.1
- net N$63: now also R11.2; no longer R14.2
- net N$66: now also J13.2; no longer J12.2
- net N$67: now also J14.2; no longer J13.2
- net N$74: now also J16.2; no longer J15.2
- net N$75: now also J17.2; no longer J16.2
- net REG_5V: now also R10.1; no longer R13.1
- net RXD: now also J4.3; no longer J9-3.S
- net SCK: now also J3.3; no longer J10.3
- net SCK_3.3V: now also J6.SCLK; no longer J4.SCLK
- net SERVO: now also J1-3.S; no longer J7-3.S
- net TOUCH1: now also J10.1, J11.Y1; no longer J2.Y1
- net TOUCH2: now also J10.2, J11.X2; no longer J2.X2
- net TOUCH3: now also J10.3, J11.Y2; no longer J2.Y2
- net TOUCH4: now also J10.4, J11.X1; no longer J2.X1
- net TXD: now also J4.4; no longer J9-4.S
- net VDD: now also J6.VDD; no longer J4.VDD
- net X_HOME: now also J9-2.1, R17.1; no longer J1-2.S, R8.1
- net Y_HOME: now also J9-4.1, R18.1; no longer J1-4.S, R9.1
- net Z_DIR: now also J2-4.1; no longer J8-4.S
- net Z_HOME: now also J9-6.1, R19.1; no longer J1-6.S, R10.1
- net Z_STEP: now also J2-5.1; no longer J8-5.S
Other:
- note added: "0R25 resistors: CSRN2010FKR250CT-ND"
- moved on the sheet: C13, C14, C15, C16, C17, C18, C19, C20, C21, C22, C23, C24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

Commit message: foo
Parts:
- R32, R33: value 0.25R 1W -> 0.20Ω 1W
- R46, R47: value 0.2R 1W -> 0.20Ω 1W
Other:
- note added: "CSRN2010FKR200CT-ND"
- note removed: "0R25 resistors: CSRN2010FKR250CT-ND"
- note removed: "989-1049-1-ND"
Changed lines of the file:
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@@
 <setting verticaltext="up"/>
 </settings>
-<grid distance="0.1" unitdist="inch" unit="inch" style="lines" multiple="1" display="yes" altdistance="0.01" altunitdist="inch" altunit="inch"/>
+<grid distance="0.1" unitdist="inch" unit="inch" style="lines" multiple="1" display="no" altdistance="0.01" altunitdist="inch" altunit="inch"/>
 <layers>
 <layer number="1" name="Top" color="4" fill="1" visible="no" active="no"/>
@@
 <part name="C17" library="freetronics-master-v1" deviceset="CAP" device="0603" value="1nF"/>
 <part name="VR2" library="pot" deviceset="TRIM_EU-" device="CT6" value="10K"/>
-<part name="R32" library="rcl" deviceset="R-EU_" device="R2010" value="0.25R 1W"/>
+<part name="R32" library="rcl" deviceset="R-EU_" device="R2010" value="0.20Ω 1W"/>
 <part name="R27" library="freetronics-master-v1" deviceset="RESISTOR" device="0603" value="47K"/>
 <part name="C18" library="freetronics-master-v1" deviceset="CAP" device="0603" value="1nF"/>
@@
 <part name="C14" library="freetronics-master-v1" deviceset="CAP" device="0603" value="220nF"/>
 <part name="C16" library="freetronics-master-v1" deviceset="CAP" device="0603" value="220nF"/>
-<part name="R33" library="rcl" deviceset="R-EU_" device="R2010" value="0.25R 1W"/>
+<part name="R33" library="rcl" deviceset="R-EU_" device="R2010" value="0.20Ω 1W"/>
 <part name="C13" library="rcl" deviceset="CPOL-EU" device="E2.5-6" value="100uF"/>
 <part name="IC7" library="eje-components" deviceset="DRV8811" device=""/>
@@
 <part name="C29" library="freetronics-master-v1" deviceset="CAP" device="0603" value="1nF"/>
 <part name="VR3" library="pot" deviceset="TRIM_EU-" device="CT6" value="10 k"/>
-<part name="R46" library="rcl" deviceset="R-EU_" device="R2010" value="0.2R 1W"/>
+<part name="R46" library="rcl" deviceset="R-EU_" device="R2010" value="0.20Ω 1W"/>
 <part name="R41" library="freetronics-master-v1" deviceset="RESISTOR" device="0603" value="47K"/>
 <part name="C30" library="freetronics-master-v1" deviceset="CAP" device="0603" value="1nF"/>
@@
 <part name="C26" library="freetronics-master-v1" deviceset="CAP" device="0603" value="220nF"/>
 <part name="C28" library="freetronics-master-v1" deviceset="CAP" device="0603" value="220nF"/>
-<part name="R47" library="rcl" deviceset="R-EU_" device="R2010" value="0.2R 1W"/>
+<part name="R47" library="rcl" deviceset="R-EU_" device="R2010" value="0.20Ω 1W"/>
 <part name="C25" library="rcl" deviceset="CPOL-EU" device="E2.5-6" value="100uF"/>
 <part name="U$106" library="freetronics-luke" deviceset="GND" device=""/>
@@
 <text x="144.78" y="226.06" size="1.27" layer="98">0603</text>
 <text x="177.8" y="226.06" size="1.27" layer="98">2010</text>
-<text x="177.8" y="215.9" size="1.27" layer="98">0R25 resistors: CSRN2010FKR250CT-ND</text>
 <text x="203.2" y="226.06" size="1.27" layer="98">2010</text>
 <text x="190.5" y="226.06" size="1.27" layer="98">0603</text>
@@
 <text x="144.78" y="53.34" size="1.27" layer="98">0603</text>
 <text x="177.8" y="53.34" size="1.27" layer="98">2010</text>
-<text x="170.18" y="50.8" size="1.27" layer="98">989-1049-1-ND</text>
+<text x="190.5" y="43.18" size="1.27" layer="98">CSRN2010FKR200CT-ND</text>
 <text x="203.2" y="53.34" size="1.27" layer="98">2010</text>
 <text x="190.5" y="53.34" size="1.27" layer="98">0603</text>
@@
 <text x="129.54" y="111.76" size="1.27" layer="98">0603</text>
 <text x="220.98" y="127" size="1.27" layer="98">C25: 399-6104-ND</text>
+<text x="190.5" y="215.9" size="1.27" layer="98">CSRN2010FKR200CT-ND</text>
 </plain>
 <instances>

Commit message: foo
Parts:
- C10, C4, C5, C7, C8: value 100 nF -> 100nF
- C2: value 47 uF -> 47µF
- C3: value 100 pF -> 100pF
- C6: value 10uF -> 10µF
- C9: value 1 uF -> 1µF
- IC3: value LD1117S33 -> LD111733
- J8: value USB-FT -> USB
- LED8: value SD act -> SD
- R8: value 0.2 ohms -> 0.2Ω
- VR1, VR3: value 10 k -> 10kΩ
- VR2: value 10K -> 10kΩ
Changed lines of the file:
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@@
 <?xml version="1.0" encoding="utf-8"?>
 <!DOCTYPE eagle SYSTEM "eagle.dtd">
-<eagle version="6.2">
+<eagle version="6.3">
 <drawing>
 <settings>
@@
 <part name="J7" library="freetronics-luke" deviceset="SJ" device="" value="HWB"/>
 <part name="U$28" library="freetronics-luke" deviceset="GND" device=""/>
-<part name="J8" library="freetronics-luke" deviceset="USB-FT" device=""/>
+<part name="J8" library="freetronics-luke" deviceset="USB-FT" device="" value="USB"/>
 <part name="Z1" library="freetronics-luke" deviceset="PGB102ST23" device=""/>
 <part name="U$66" library="freetronics-luke" deviceset="GND" device=""/>
@@
 <part name="LED5" library="freetronics-master-v1" deviceset="LED" device="0603" value="Y"/>
 <part name="U$85" library="freetronics-luke" deviceset="GND" device=""/>
-<part name="IC3" library="burr-brown" deviceset="REG1117" device="" value="LD1117S33"/>
+<part name="IC3" library="burr-brown" deviceset="REG1117" device="" value="LD111733"/>
 <part name="P+22" library="supply1" deviceset="+5V" device=""/>
 <part name="IC1" library="40xx" deviceset="4050" device="D" value="HEF4050B"/>
@@
 <part name="P+14" library="supply1" deviceset="+5V" device=""/>
 <part name="P+15" library="supply1" deviceset="+5V" device=""/>
-<part name="C4" library="freetronics-master-v1" deviceset="CAP" device="0603" value="100 nF"/>
+<part name="C4" library="freetronics-master-v1" deviceset="CAP" device="0603" value="100nF"/>
 <part name="P+16" library="supply1" deviceset="+5V" device=""/>
-<part name="VR1" library="pot" deviceset="TRIM_EU-" device="CT6" value="10 k"/>
+<part name="VR1" library="pot" deviceset="TRIM_EU-" device="CT6" value="10kΩ"/>
 <part name="IC2" library="SparkFun" deviceset="MC34063" device="SMD" value="MC34063"/>
-<part name="C3" library="freetronics-master-v1" deviceset="CAP" device="0603" value="100 pF"/>
+<part name="C3" library="freetronics-master-v1" deviceset="CAP" device="0603" value="100pF"/>
 <part name="C1" library="rcl" deviceset="CPOL-EU" device="E2.5-6" value="100uF"/>
 <part name="L1" library="SparkFun" deviceset="INDUCTOR" device="CR75" value="33 uH"/>
-<part name="C2" library="rcl" deviceset="C-EU" device="C1210" value="47 uF"/>
+<part name="C2" library="rcl" deviceset="C-EU" device="C1210" value="47µF"/>
 <part name="P+11" library="supply1" deviceset="+12V" device=""/>
 <part name="LED7" library="freetronics-master-v1" deviceset="LED" device="0603" value="12"/>
@@
 <part name="R9" library="freetronics-master-v1" deviceset="RESISTOR" device="0603" value="1k"/>
 <part name="R10" library="freetronics-master-v1" deviceset="RESISTOR" device="0603" value="3k0"/>
-<part name="R8" library="rcl" deviceset="R-EU_" device="R1210" value="0.2 ohms"/>
+<part name="R8" library="rcl" deviceset="R-EU_" device="R1210" value="0.2Ω"/>
 <part name="R12" library="freetronics-master-v1" deviceset="RESISTOR" device="0603" value="22R"/>
 <part name="R17" library="freetronics-master-v1" deviceset="RESISTOR" device="0603" value="10k"/>
@@
 <part name="R11" library="freetronics-master-v1" deviceset="RESISTOR" device="0603" value="1k"/>
 <part name="R13" library="freetronics-master-v1" deviceset="RESISTOR" device="0603" value="10k"/>
-<part name="LED8" library="freetronics-master-v1" deviceset="LED" device="0603" value="SD act"/>
+<part name="LED8" library="freetronics-master-v1" deviceset="LED" device="0603" value="SD"/>
 <part name="P+3" library="supply1" deviceset="+5V" device=""/>
 <part name="D2" library="freetronics-luke" deviceset="SCHOTTKY" device="" value="CDBA120"/>
@@
 <part name="U$44" library="freetronics-luke" deviceset="GND" device=""/>
 <part name="U$45" library="freetronics-luke" deviceset="GND" device=""/>
-<part name="C5" library="freetronics-master-v1" deviceset="CAP" device="0603" value="100 nF"/>
-<part name="C6" library="freetronics-master-v1" deviceset="CAP" device="0805" value="10uF"/>
+<part name="C5" library="freetronics-master-v1" deviceset="CAP" device="0603" value="100nF"/>
+<part name="C6" library="freetronics-master-v1" deviceset="CAP" device="0805" value="10µF"/>
 <part name="R14" library="freetronics-master-v1" deviceset="RESISTOR" device="0603" value="10k"/>
 <part name="R16" library="freetronics-master-v1" deviceset="RESISTOR" device="0603" value="22R"/>
@@
 <part name="R26" library="freetronics-master-v1" deviceset="RESISTOR" device="0603" value="47K"/>
 <part name="C17" library="freetronics-master-v1" deviceset="CAP" device="0603" value="1nF"/>
-<part name="VR2" library="pot" deviceset="TRIM_EU-" device="CT6" value="10K"/>
+<part name="VR2" library="pot" deviceset="TRIM_EU-" device="CT6" value="10kΩ"/>
 <part name="R32" library="rcl" deviceset="R-EU_" device="R2010" value="0.20Ω 1W"/>
 <part name="R27" library="freetronics-master-v1" deviceset="RESISTOR" device="0603" value="47K"/>
@@
 <part name="R40" library="freetronics-master-v1" deviceset="RESISTOR" device="0603" value="47K"/>
 <part name="C29" library="freetronics-master-v1" deviceset="CAP" device="0603" value="1nF"/>
-<part name="VR3" library="pot" deviceset="TRIM_EU-" device="CT6" value="10 k"/>
+<part name="VR3" library="pot" deviceset="TRIM_EU-" device="CT6" value="10kΩ"/>
 <part name="R46" library="rcl" deviceset="R-EU_" device="R2010" value="0.20Ω 1W"/>
 <part name="R41" library="freetronics-master-v1" deviceset="RESISTOR" device="0603" value="47K"/>
@@
 <part name="U$106" library="freetronics-luke" deviceset="GND" device=""/>
 <part name="J5" library="SparkFun" deviceset="POWER_JACK" device="SLT" value="12V Supply"/>
-<part name="C7" library="freetronics-master-v1" deviceset="CAP" device="0603" value="100 nF"/>
-<part name="C8" library="freetronics-master-v1" deviceset="CAP" device="0603" value="100 nF"/>
-<part name="C10" library="freetronics-master-v1" deviceset="CAP" device="0603" value="100 nF"/>
+<part name="C7" library="freetronics-master-v1" deviceset="CAP" device="0603" value="100nF"/>
+<part name="C8" library="freetronics-master-v1" deviceset="CAP" device="0603" value="100nF"/>
+<part name="C10" library="freetronics-master-v1" deviceset="CAP" device="0603" value="100nF"/>
 <part name="C12" library="freetronics-master-v1" deviceset="CAP" device="0603" value="22pF"/>
 <part name="C11" library="freetronics-master-v1" deviceset="CAP" device="0603" value="22pF"/>
-<part name="C9" library="freetronics-master-v1" deviceset="CAP" device="0603" value="1 uF"/>
+<part name="C9" library="freetronics-master-v1" deviceset="CAP" device="0603" value="1µF"/>
 <part name="J10" library="pinhead" deviceset="PINHD-1X4" device="" value="Touchscreen"/>
 <part name="J4" library="pinhead" deviceset="PINHD-1X4" device="" value="UART"/>

Commit message: added reset button
Parts:
- added S1: RESET, freetronics-master-v1:TAC_SWITCH_2PIN
Connections:
- net !RESET: now also S1.S
- net GND: now also S1.P
Other:
- moved on the sheet: C1, C10, C11, C12, C13, C14, C15, C16, C17, C18, C19, C2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
